File: kicad-project/clock_top.sch (KiCad schematic (older format))
At the start: 53 parts, among them SW1 PEC16, U1 ZS-042, U2 ZS-040, U3 KPC452, U4 KPC452, U5 KPC452, U6 KPC452

Commit message: git repo refactor: v2 in12, 6 tubes, arduino
Parts:
- removed R20: 2.2K, Resistor_SMD:R_0805_2012Metric_Pad1.15x1.40mm_HandSolder, symbol Device:R
- removed U2: ZS-040, clock:zs-040, symbol custom_library:ZS-040
- removed U3, U4, U5, U6: KPC452, Package_SO:SO-4_4.4x3.6mm_P2.54mm, symbol Isolator:LTV-352T
- added C11: 100nF, 250V, Capacitor_SMD:C_1206_3216Metric_Pad1.42x1.75mm_HandSolder, symbol Device:C
- added C8: 100nF, 50V, Capacitor_SMD:C_0805_2012Metric_Pad1.15x1.40mm_HandSolder, symbol Device:C
- added D6: HV5812, Package_SO:SOIC-28W_7.5x17.9mm_P1.27mm, symbol clock_top-rescue:HV5812-custom_library
- added LL5, LL6: IN-12B, v2:IN12-HI_IE, symbol clock_top-rescue:IN-12B-custom_library
- D1: symbol custom_library:MAX1771 -> clock_top-rescue:MAX1771-custom_library
- D4, D5: symbol custom_library:HV5812 -> clock_top-rescue:HV5812-custom_library
- L1: symbol custom_library:B82477R4224M100 -> clock_top-rescue:B82477R4224M100-custom_library
- LL1, LL2, LL3, LL4: footprint clock:PL31 -> v2:IN12-HI_IE; symbol custom_library:IN-12B -> clock_top-rescue:IN-12B-custom_library
- R17: value 2.2K -> 150K
- R18, R19: value 2.2K -> 22K
- U1: symbol custom_library:ZS-042 -> clock_top-rescue:ZS-042-custom_library
- VD1: symbol custom_library:ES2J -> clock_top-rescue:ES2J-custom_library
- VT1: symbol custom_library:STD18N55M5 -> clock_top-rescue:STD18N55M5-custom_library
Connections:
- net +5V: now also C8.2, D6.28 (VDD)
- net CLOCK: now also A1.25 (D10), D6.15 (CLOCK); no longer A1.27 (D12)
- net DATA: now also A1.27 (D12), D4.27 (Data_In); no longer A1.25 (D10), D5.27 (Data_In)
- net GND: now also R17.1, C11.2, C8.1, D6.13 (BLANKING), D6.14 (GND)
- net HV: now also R18.2, R19.2
- net HV_C: now also R17.2, C11.1, D6.1 (VPP)
- net SHUT: no longer A1.19 (D4)
- net STROBE: now also D6.16 (STROBE)
- net at D4.2 (Data_Out): now also D5.27 (Data_In)
- net at D5.2 (Data_Out): now also D6.27 (Data_In); no longer D4.27 (Data_In)
- net at R18.1: now also LL5.1 (A)
- net at R19.1: now also LL6.1 (A)
- net RT_INT: no longer names the net of A1.22 (D7)
- net RT_INT: no longer U1.2 (SQW)
- net RxD: no longer names the net of A1.15 (D0/RX)
- net TxD: no longer names the net of A1.16 (D1/TX)
- net _1-.: no longer names the net of A1.20 (D5)
- net _1-.: no longer R17.2
- net _2-.: no longer names the net of A1.21 (D6)
- net _2-.: no longer R18.2
- net _3-.: no longer names the net of A1.23 (D8)
- net _3-.: no longer R19.2
- net _4-.: no longer names the net of A1.24 (D9)
- new net 5-.: LL5.12 (.)
- new net 5-0: D6.23 (HVOUT4), LL5.2 (0)
- new net 5-1: D6.3 (HVOUT20), LL5.11 (1)
- new net 5-2: D6.4 (HVOUT19), LL5.10 (2)
- new net 5-3: D6.5 (HVOUT18), LL5.9 (3)
- new net 5-4: D6.6 (HVOUT17), LL5.8 (4)
- new net 5-5: D6.7 (HVOUT16), LL5.7 (5)
- new net 5-6: D6.8 (HVOUT15), LL5.6
- new net 5-7: D6.26 (HVOUT1), LL5.5 (7)
- new net 5-8: D6.25 (HVOUT2), LL5.4 (8)
- new net 5-9: D6.24 (HVOUT3), LL5.3 (9)
- new net 6-.: LL6.12 (.)
- new net 6-0: D6.12 (HVOUT11), LL6.2 (0)
- new net 6-1: D6.22 (HVOUT5), LL6.11 (1)
- new net 6-2: D6.21 (HVOUT6), LL6.10 (2)
- new net 6-3: D6.20 (HVOUT7), LL6.9 (3)
- new net 6-4: D6.19 (HVOUT8), LL6.8 (4)
- new net 6-5: D6.18 (HVOUT9), LL6.7 (5)
- new net 6-6: D6.17 (HVOUT10), LL6.6
- new net 6-7: D6.9 (HVOUT14), LL6.5 (7)
- new net 6-8: D6.10 (HVOUT13), LL6.4 (8)
- new net 6-9: D6.11 (HVOUT12), LL6.3 (9)
Other:
- moved on the sheet: LL3, LL4, R12, R13, R9
