File: kicad-projects/in12-nixie-shield/clock_top.kicad_pcb (KiCad board)
At the start: 2 copper layers, 158 x 54 mm, 67 parts, among them J1 Conn_01x01_Male, J2 Conn_01x01_Male, J3 Conn_01x01_Male, J4 Conn_01x01_Male, SW1 PEC16, U2 MAX1771xSA, U4 KPC452, U5 KPC452

Commit message: pcb: revision bump
stm32f103: revison 2
  - added: D+ to +5V (fixed error: unable to enumerate device)
  - added: usb phy int pin pull up to +3.3v (fixed no irq from phy)
  - moved: JTAG connector is moved to bottom layer

clock-top (nixie shild): revision 1, initial version

removed pf-info-cache (temp kicad file)
Parts:
- C11: footprint Capacitor_SMD:C_1206_3216Metric_Pad1.42x1.75mm_HandSolder -> Capacitor_SMD:C_1206_3216Metric_Pad1.33x1.80mm_HandSolder
- moved D4 4.45 mm to (139.6, 112.0)
Other:
- rule pad_to_mask_clearance: 0.051 -> 0
- board text added: "+3.3V"
- board text added: "+5V"
- board text added: "+VIN"
- board text added: "A"
- board text added: "B"
- board text added: "CLOCK"
- board text added: "DATA"
- board text added: "GND"
- board text added: "SHUT"
- board text added: "STROBE"
- board text added: "SW"
- board text added: "X"
- board text added: "_2."
- board text added: "_4."
- board text added: "arduino NIXIE shield rev. 1"
