File: kicad-projects/in12-nixie-shield/clock_top.kicad_sch (KiCad schematic)
At the start: 63 parts, among them J1 Conn_01x01_Male, J2 Conn_01x01_Male, J3 Conn_01x01_Male, J4 Conn_01x01_Male, SW1 PEC16, U2 MAX1771xSA, U4 KPC452, U5 KPC452

Commit message: pcb: revision bump
stm32f103: revison 2
  - added: D+ to +5V (fixed error: unable to enumerate device)
  - added: usb phy int pin pull up to +3.3v (fixed no irq from phy)
  - moved: JTAG connector is moved to bottom layer

clock-top (nixie shild): revision 1, initial version

removed pf-info-cache (temp kicad file)
Parts:
- C11: footprint Capacitor_SMD:C_1206_3216Metric_Pad1.42x1.75mm_HandSolder -> Capacitor_SMD:C_1206_3216Metric_Pad1.33x1.80mm_HandSolder
Changed lines of the file:
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@@
       (effects (font (size 1.27 1.27)) (justify left))
     )
-    (property "Footprint" "Capacitor_SMD:C_1206_3216Metric_Pad1.42x1.75mm_HandSolder" (id 2) (at 307.34 178.7652 0)
+    (property "Footprint" "Capacitor_SMD:C_1206_3216Metric_Pad1.33x1.80mm_HandSolder" (id 2) (at 307.34 178.7652 0)
       (effects (font (size 1.27 1.27)) hide)
     )
@@
     )
     (path "/00000000-0000-0000-0000-00005f0f2794"
-      (reference "C11") (unit 1) (value "100nF, 250V") (footprint "Capacitor_SMD:C_1206_3216Metric_Pad1.42x1.75mm_HandSolder")
+      (reference "C11") (unit 1) (value "100nF, 250V") (footprint "Capacitor_SMD:C_1206_3216Metric_Pad1.33x1.80mm_HandSolder")
     )
     (path "/69adf70b-0663-412c-aa45-16e6e15c090d"
