File: kicad-projects/stm32f103/stm32f103.kicad_pcb (KiCad board)
At the start: 2 copper layers, 68.6 x 53.3 mm, 68 parts, among them J1 Conn_01x20_Male, J2 USB_C_Receptacle, J3 Jack-DC, J4 Conn_02x02_Odd_Even, J5 Conn_01x10_Female, J6 Conn_01x06_Female, J7 Conn_01x08_Female, J8 Conn_01x08_Female, SW1 SW_Push, U1 TPS62175DQC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

Commit message: pcb: revision bump
stm32f103: revison 2
  - added: D+ to +5V (fixed error: unable to enumerate device)
  - added: usb phy int pin pull up to +3.3v (fixed no irq from phy)
  - moved: JTAG connector is moved to bottom layer

clock-top (nixie shild): revision 1, initial version

removed pf-info-cache (temp kicad file)
Parts:
- added Q1: IRLML6401, Package_TO_SOT_SMD:SOT-23, F.Cu at (149.5, 66.2)
- added R29: 2.1K, Resistor_SMD:R_0805_2012Metric_Pad1.20x1.40mm_HandSolder, F.Cu at (168.0, 59.5)
- added R30: 1.5K, Resistor_SMD:R_0805_2012Metric_Pad1.20x1.40mm_HandSolder, F.Cu at (149.2, 63.2)
- J1: moved to B.Cu
- moved U5 7.80 mm to (118.2, 63.4)
- moved R19 3.59 mm to (121.8, 59.5), turned to -90 degrees
- moved R5 2.85 mm to (172.0, 77.8)
- moved J1 2.61 mm to (141.0, 91.0), turned to 0 degrees
- moved C17 2.14 mm to (121.0, 63.5), turned to -90 degrees
- moved C18 1.48 mm to (124.1, 59.5), turned to -90 degrees
- moved U4 1.00 mm to (125.5, 64.5)
- moved R6 0.99 mm to (148.2, 83.9)
- moved C11 0.50 mm to (152.7, 69.5)
- moved R18 0.43 mm to (126.6, 59.5)
- moved R17 0.35 mm to (128.8, 59.5)
- moved C15 0.25 mm to (164.2, 67.0), turned to -90 degrees
- moved D2 0.25 mm to (122.2, 74.8)
- moved R25 0.16 mm to (155.1, 59.5)
- moved R13 0.15 mm to (120.0, 66.9)
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Connections:
- R15 pad 1: /D5 -> +5V
- R15 pad 2: +5V -> /D5
- R16 pad 1: /D10 -> +5V
- R16 pad 2: +5V -> /D10
- U3 pad 14: /D2 -> /ÌNT_PHY
- U3 pad 15: /D3 -> /D2
- U3 pad 16: /D4 -> /D3
- U3 pad 17: /D5 -> /D4
- U3 pad 18: /ÌNT_PHY -> /D5
- U3 pad 19: unconnected-(U3-Pad19) -> /D6
- U3 pad 25: /D6 -> /D7
- U3 pad 26: /D7 -> /D8
- U3 pad 27: /D8 -> /D9
- U3 pad 28: /D9 -> /D10
- U3 pad 29: /D10 -> /USB_EN
Routing:
- net GND: track 159.9 -> 130.1 mm, vias 31 -> 36
- net /ÌNT_PHY: track 84.9 -> 70.9 mm
- net /USB_EN: track 0.00 -> 13.8 mm
- net /D6: track 19.1 -> 31.6 mm
- net /D+: track 25.9 -> 13.8 mm, vias 0 -> 2
- net /CC2: track 32.3 -> 25.0 mm
- net VBUS: track 23.2 -> 28.9 mm, vias 2 -> 4
- net /JTDI: track 23.1 -> 28.1 mm
- net +3.3V: track 181.3 -> 186.1 mm, vias 9 -> 8
- net /NJTRST: track 23.8 -> 28.4 mm
- net Net-(J1-Pad11): track 7.43 -> 3.30 mm
- net /JTCK / SWCLK: track 19.5 -> 23.4 mm
- net /NRTS: track 65.9 -> 69.5 mm
- net /ADC12_IN0: track 35.8 -> 32.2 mm
- net /D-: track 16.4 -> 12.9 mm
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Other:
- board text added: "BOOT modes: 0 user flash 1 system memory"
- board text added: "STM32F103 UNO R3 rev.2"
- board text removed: "BOOT modes: 0 user flash(default) 1 system memory"
- board text removed: "STM32F103 UNO R3 rev.1"
